File: BusinessCard.kicad_sch (KiCad schematic)
At the start: 59 parts, among them J1 RST, J2 USB_B_Micro, SW1 SW_Push, SW10 SW_Push, SW11 SW_Push, SW12 SW_Push, SW13 SW_Push, SW14 SW_Push, SW15 SW_Push, SW16 SW_Push, SW2 SW_Push, SW3 SW_Push, SW4 SW_Push, SW5 SW_Push, SW6 SW_Push, SW7 SW_Push, SW8 SW_Push, SW9 SW_Push, U2 USBLC6-2SC6, U3 ATmega32U4-M, Y1 X322516MLB4SI

Commit message: Updated to the current revision
Parts:
- removed J2: USB_B_Micro, Connector_USB:USB_Micro-B_XKB_U254-051T-4BH83-F1S, symbol Connector:USB_B_Micro
- added C6: 1uF, Capacitor_SMD:C_0603_1608Metric, symbol Device:C_Small
- added J3: USB_C_Receptacle_USB2.0_14P, Connector_USB:USB_C_Receptacle_G-Switch_GT-USB-7010ASV, symbol Connector:USB_C_Receptacle_USB2.0_14P
- added R2, R3: 22ohm, Resistor_SMD:R_0402_1005Metric, symbol Device:R_Small
- added R4, R5: 5.1k, Resistor_SMD:R_0402_1005Metric, symbol Device:R_Small
- C1, C2: LCSC (none) -> C32949
- C3, C4, C5: LCSC (none) -> C1525
- D1, D10, D11, D12, D13, D14, D15, D16, D2, D3, D4, D5, D6, D7, D8, D9: value SOD-123 -> SOD-323; LCSC (none) -> C2128
- D18, D19, D20, D21, D22, D23, D24, D25, D26, D27, D28, D29, D30, D31, D32, D33: LCSC (none) -> C965555; now not fitted
- J1: now not fitted
- R1: LCSC (none) -> C25744
- SW1, SW10, SW11, SW12, SW13, SW14, SW15, SW16, SW2, SW3, SW4, SW5, SW6, SW7, SW8, SW9: LCSC (none) -> C318884
- U2: LCSC (none) -> C2827654
- U3: LCSC (none) -> C112161
- Y1: LCSC (none) -> C13738
Connections:
- net +5V: now also J3.A4 (VBUS), J3.A9 (VBUS), J3.B4 (VBUS), J3.B9 (VBUS)
- net GND: now also C6.2, J3.A1 (GND), J3.A12 (GND), J3.B1 (GND), J3.B12 (GND), J3.S1 (SHIELD), R4.2, R5.1
- net USBLC6_DN: now also R3.1
- net USBLC6_DP: now also R2.1
- net USB_UCAP: now also C6.1
- new net: J3.A7 (D-), J3.B7 (D-), R3.2
- new net: J3.B5 (CC2), R5.2
- new net: J3.A5 (CC1), R4.1
- new net: J3.A6 (D+), J3.B6 (D+), R2.2
- no-connect marks 3 -> 19
Other:
- moved on the sheet: U2

Commit message: Update
Connections:
- net +5V: now also D18.4 (VDD), D19.4 (VDD), D20.4 (VDD), D21.4 (VDD), D22.4 (VDD), D23.4 (VDD), D24.4 (VDD), D25.4 (VDD), D26.4 (VDD), D27.4 (VDD), D28.4 (VDD), D29.4 (VDD), D30.4 (VDD), D31.4 (VDD), D32.4 (VDD), D33.4 (VDD)
- net USBLC6_DN: now also U2.3 (I/O2); no longer U2.6 (I/O1)
- net USB_DP: now also U2.6 (I/O1); no longer U2.3 (I/O2)
Other:
- moved on the sheet: D18, D19, D20, D21, D22, D23, D24, D25, D26, D27, D28, D29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
